Commit message: Gerçekçi çarpışma fiziği + ön kama görsel düzeltmesi
Fizik modeli (URDF + sim_engine):
- Ön kama artık gerçek bir collider: yatayla ~22°, ön ucu yerden 0.5 mm,
  arkası gövdeye gömülü çelik rampa → rakibin altına girip kaldırır
- URDF CoM merkezli çerçeveye taşındı (PyBullet base_link çerçevesini
  CoM'e oturtuyor): CoM yerden ~21 mm, tekerlek aksının 10 mm önünde,
  ağırlığın %70'i tahrikli tekerleklerde, %30 kızakta
- Kütle muhasebesi: gövde dışı linkler (kama/tekerlek/kızak/sensör)
  düşülerek toplam kütle paneldeki değere tam eşitlenir; atalet de
  kütleyle orantılı ölçeklenir
- Malzemeler: gövde μ=0.62 e=0.03, tekerlek μ=1.2 + yuvarlanma direnci,
  kızak μ=0.06 + anizotropik (ileri kayar/yana direnir), kama μ=0.10
  + anizotropik (rampa yönünde daha kaygan)
- Çözücü: 120 iterasyon, koni sürtünmesi, split impulse, 240 Hz
- Temas modeli: robot-robot temas kuvveti telemetrisi + plastik kayıp
  (yaklaşma hızının %6'sı sönümlenir) → kinetik enerjinin >%95'i kaybolur
- Motor: jSumo Force Up 6V tork/hız değerleri; itme kuvveti zemin
  tutunmasıyla sınırlanır → ağır robot hafifi iter

Görsel (index.html):
- Bıçak, dik plaka yerine gerçek kama (üçgen prizma) olarak yeniden
  modellendi: yere yakın keskin ön uç, arkada 3.5 mm kalınlık
- Tüm parçalar yeni CoM çerçevesine taşındı, tekerlek aksı hizalandı
- Takım rengi zemin halkası yanlış eksende dikey duruyordu → yatık
- Telemetriye 'Çarpışma kuvveti' satırı eklendi

Oda/paylaşım:
- Hakem kopuksa bayat oda devralınabilir (terk edilmiş oda kilidi önlendi)
- smoke_test açık mod kontrolü + tests/physics_test.py eklendi
- README: fizik/çarpışma modeli bölümü

File: sim/urdf/mini_sumo_bot.urdf (robot description, URDF)
Before this commit: robot mini_sumo_bot, 8 links, 7 joints
Links:
- added link blade, mass 0.024; collision box size=0.026 0.092 0.0035; visual box size=0.026 0.092 0.0035
- link base_link: mass 0.5 -> 0.461; geometry collision box size=0.058 0.068 0.036; collision box size=0.092 0.070 0.017
- link e3z_left: mass 0.0005 -> 0.001; geometry collision box size=0.016 0.010 0.010; visual box size=0.016 0.010 0.010
- link e3z_right: mass 0.0005 -> 0.001; geometry collision box size=0.016 0.010 0.010; visual box size=0.016 0.010 0.010
- link left_wheel: mass 0.001 -> 0.004
- link right_wheel: mass 0.001 -> 0.004
- link skid: mass 0.0005 -> 0.004
Joints:
- added joint blade_joint: type fixed, parent base_link, child blade, origin xyz=0.038 0 -0.0137 rpy=0 0 0
- joint e3z_left_joint: origin xyz=0.047 0.022 0.004 rpy=0 0 0 -> xyz=0.030 0.021 0.0218 rpy=0 0 0
- joint e3z_right_joint: origin xyz=0.047 -0.022 0.004 rpy=0 0 0 -> xyz=0.030 -0.021 0.0218 rpy=0 0 0
- joint left_wheel_joint: origin xyz=-0.018 0.036 -0.008 rpy=1.5708 0 0 -> xyz=-0.010 0.036 0.000 rpy=1.5708 0 0
- joint qtr_left_joint: origin xyz=0.030 0.028 -0.014 rpy=0 0 0 -> xyz=0.028 0.026 -0.0107 rpy=0 0 0
- joint qtr_right_joint: origin xyz=0.030 -0.028 -0.014 rpy=0 0 0 -> xyz=0.028 -0.026 -0.0107 rpy=0 0 0
- joint right_wheel_joint: origin xyz=-0.018 -0.036 -0.008 rpy=1.5708 0 0 -> xyz=-0.010 -0.036 0.000 rpy=1.5708 0 0
- joint skid_joint: origin xyz=0.038 0 -0.0245 rpy=0 0 0 -> xyz=0.030 0 -0.0158 rpy=0 0 0
